Commit message: implementacion de cinematica directa. falta agregar articulacion prismatica

File: robot_description/urdf/robot_description.urdf (robot description, URDF)
Before this commit: robot edo, 7 links, 6 joints
Joints:
- joint joint_1: origin xyz=0.057188 0.0059831 0.13343 rpy=1.5708 6.9389E-16 -3.1416 -> xyz=0.0 0.0 0.13343 rpy=1.571 0.0 -3.1416
- joint joint_5: origin xyz=0 0 -0.1053 rpy=3.1416 1.1102E-14 3.1416 -> xyz=0 0 -0.1053 rpy=3.14159 0 3.14159
- joint joint_6: origin xyz=-0.0039 0 0.1636 rpy=-1.5708 1.249E-14 0 -> xyz=-0.0039 0 0.1636 rpy=-1.5708 0 0

Commit message: eslabon y art. extra. corregir dh, control cinematico y pulir urdf

File: robot_description/urdf/robot_description.urdf (robot description, URDF)
Before this commit: robot edo, 7 links, 6 joints
Links:
- added link cylinder_link, mass 1.0; collision cylinder length=0.25 radius=0.03; visual cylinder length=0.25 radius=0.03
Joints:
- added joint prismatic_joint: type prismatic, parent link_3, child cylinder_link, origin xyz=0 0 0.0 rpy=0 0 0, axis 0 -1 0, limit lower=0.0 upper=0.5 effort=50 velocity=1.0
- joint joint_4: parent link_3 -> cylinder_link

Commit message: Update_robot_description.urdf

File: robot_description/urdf/robot_description.urdf (robot description, URDF)
Before this commit: robot edo, 8 links, 7 joints
Links:
- link cylinder_link: geometry collision cylinder length=0.25 radius=0.033; visual cylinder length=0.25 radius=0.033
Joints:
- joint joint_1: origin xyz=0.0 0.0 0.13343 rpy=1.571 0.0 -3.1416 -> xyz=0.06 0.0 0.084 rpy=1.571 0.0 -3.1416
- joint joint_2: limit (none) -> lower=0 upper=1.10 effort=50 velocity=1.0; type continuous -> revolute
- joint joint_3: limit (none) -> lower=0 upper=1.5 effort=50 velocity=1.0; type continuous -> revolute
- joint joint_4: origin xyz=0.0088 -0.1588 0 rpy=-1.5708 0 0 -> xyz=0 -0.121 0 rpy=-1.5708 0 0
- joint joint_5: limit (none) -> lower=-1.5 upper=1.5 effort=50 velocity=1.0; type continuous -> revolute
- joint prismatic_joint: limit lower=0.0 upper=0.5 effort=50 velocity=1.0 -> lower=0.2 upper=0.3 effort=50 velocity=1.0; origin xyz=0 0 0.0 rpy=0 0 0 -> xyz=0.01 0 0 rpy=0 0 0
